File: Flash-2716.kicad_sch (KiCad schematic)
At the start: 12 parts, among them J1 Conn_01x12, J2 Conn_01x12, U1 SST39SF010

Commit message: Add 2716 socket & storage
Parts:
- added C1: Jumper_3_Open, Connector_PinHeader_2.54mm:PinHeader_1x03_P2.54mm_Vertical, symbol Jumper:Jumper_3_Open
- added J3, J4: 2716, Package_DIP:DIP-24_W15.24mm_Socket, symbol MBC-1000_Mainboard:2716
Connections:
- net A0: now also J3.8 (A0)
- net A1: now also J3.7 (A1)
- net A10: now also J3.19 (A10)
- net A2: now also J3.6 (A2)
- net A3: now also J3.5 (A3)
- net A4: now also J3.4 (A4)
- net A5: now also J3.3 (A5)
- net A6: now also J3.2 (A6)
- net A7: now also J3.1 (A7)
- net A8: now also J3.23 (A8)
- net A9: now also J3.22 (A9)
- net BUS-A11: now also J3.21 (Vpp)
- net D0: now also J3.9 (Q0)
- net D1: now also J3.10 (Q1)
- net D2: now also J3.11 (Q2)
- net D3: now also J3.13 (Q3)
- net D4: now also J3.14 (Q4)
- net D5: now also J3.15 (Q5)
- net D6: now also J3.16 (Q6)
- net D7: now also J3.17 (Q7)
- net GND: now also J3.12 (GND)
- net VCC: now also J3.24 (Vcc)
- net ~{OE}: now also J3.20 (~{OE})
- net ~{CE} renamed ~{BUS-CE}
- net ~{BUS-CE}: now also C1.2 (C); no longer U1.22 (CE)
- new net ~{CE-27}: C1.1 (A), J3.18 (~{CE}/PGM)
- new net ~{CE-39}: C1.3 (B), U1.22 (CE)

Commit message: Cleanup & plot gerbers
Parts:
- renumbered J3 to J2, J4 to J3, J2 to J4
Changed lines of the file:
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@@
 		(on_board yes)
 		(dnp no)
-		(property "Reference" "J2"
+		(property "Reference" "J4"
 			(at 208.788 50.8578 0)
 			(effects
@@
 			(project "Flash-2716"
 				(path "/4f4afbba-2cb7-42f3-8560-8215f94c8e1f"
-					(reference "J2")
+					(reference "J4")
 					(unit 1)
 				)
@@
 		(dnp no)
 		(fields_autoplaced yes)
-		(property "Reference" "J3"
+		(property "Reference" "J2"
 			(at 43.18 36.83 0)
 			(do_not_autoplace yes)
@@
 			(project "Flash-2716"
 				(path "/4f4afbba-2cb7-42f3-8560-8215f94c8e1f"
-					(reference "J3")
+					(reference "J2")
 					(unit 1)
 				)
@@
 		(dnp no)
 		(fields_autoplaced yes)
-		(property "Reference" "J4"
+		(property "Reference" "J3"
 			(at 43.18 100.33 0)
 			(do_not_autoplace yes)
@@
 			(project "Flash-2716"
 				(path "/4f4afbba-2cb7-42f3-8560-8215f94c8e1f"
-					(reference "J4")
-					(unit 1)
-				)
+					(reference "J3")
+					(unit 1)
+				)
